File: pcb/wifilcd.sch (KiCad schematic (older format))
At the start: 23 parts, among them P1 CONN_01X02, P2 CONN_01X06, Q1 BSS138, U1 AP1117D33, U2 TM022HDH26, U3 ESP-12E

Commit message: Minor PCB changes
Parts:
- Q1: footprint Housings_SOT-23_SOT-143_TSOT-6:SOT-23 -> Housings:SOT-23
- U2: footprint Modules:TM022HDH26 -> Modules:TM022HDH26_PADSONLY
Changed lines of the file:
@@
 F 0 "U2" H 6275 4700 60  0000 C CNN
 F 1 "TM022HDH26" H 6175 5500 60  0000 C CNN
-F 2 "Modules:TM022HDH26" H 6025 4750 60  0001 C CNN
+F 2 "Modules:TM022HDH26_PADSONLY" H 6025 4750 60  0001 C CNN
 F 3 "" H 6025 4750 60  0000 C CNN
 	1    6125 4750
@@
 F 0 "Q1" H 7400 4451 40  0000 R CNN
 F 1 "BSS138" H 7400 4750 40  0000 R CNN
-F 2 "Housings_SOT-23_SOT-143_TSOT-6:SOT-23" H 7270 4702 29  0000 C CNN
+F 2 "Housings:SOT-23" H 7270 4702 29  0000 C CNN
 F 3 "" H 7400 4600 60  0000 C CNN
 	1    7400 4600
